Commit message: working version by Cayden

File: ur10_robotiq_85/urdf/ur10_robotiq_85.urdf.xacro (robot description, xacro)
@@ -1,6 +1,19 @@
-<robot name="ur10" xmlns:xacro="http://www.ros.org/wiki/xacro" xmlns:xi="http://www.w3.org/2001/XInclude">
-<!-- combined urdf file -->
-<xacro:include filename="$(find ur_description)/urdf/ur10_robot.urdf.xacro"/>
-<!-- add any joints/links required to connect the two -->
-<xacro:include filename="$(find robotiq_85_description)/urdf/robotiq_85_gripper.xacro" />
+<?xml version="1.0"?>
+<robot name="ur10_robotiq_85" xmlns:xacro="http://ros.org/wiki/xacro">
+	<xacro:arg name="limited" default="true"/>
+	<!-- THE ROBOT -->
+	<link name="world" />
+	<!-- UR10 -->
+	<xacro:include filename="$(find ur_description)/urdf/ur10.urdf.xacro" />
+	<joint name="world_joint" type="fixed">
+		<parent link="world" />
+		<child link = "simple_arm_base_link" />
+		<origin xyz="0.0 0.0 0.0" rpy="0.0 0.0 0.0" />
+	</joint>
+	<xacro:ur10_robot prefix="simple_arm_" joint_limited="true"/>
+	<!-- Robotiq 85-->
+	<xacro:include filename="$(find robotiq_85_description)/urdf/robotiq_85_gripper.urdf.xacro" />
+	<xacro:robotiq_85_gripper prefix="simple_gripper_" parent="simple_arm_tool0">
+		<origin xyz="0 0 0" rpy="${pi/2} -${pi/2} 0" />
+	</xacro:robotiq_85_gripper>
 </robot>

File: ur3_robotiq_85/urdf/ur3_robotiq_85.urdf.xacro (robot description, xacro)
@@ -1,6 +1,19 @@
-<robot name="ur3" xmlns:xacro="http://www.ros.org/wiki/xacro" xmlns:xi="http://www.w3.org/2001/XInclude">
-<!-- combined urdf file -->
-<xacro:include filename="$(find ur_description)/urdf/ur3_robot.urdf.xacro"/>
-<!-- add any joints/links required to connect the two -->
-<xacro:include filename="$(find robotiq_85_description)/urdf/robotiq_85_gripper.xacro" />
+<?xml version="1.0"?>
+<robot name="ur3_robotiq_85" xmlns:xacro="http://ros.org/wiki/xacro">
+	<xacro:arg name="limited" default="true"/>
+	<!-- THE ROBOT -->
+	<link name="world" />
+	<!-- UR3 -->
+	<xacro:include filename="$(find ur_description)/urdf/ur3.urdf.xacro" />
+	<joint name="world_joint" type="fixed">
+		<parent link="world" />
+		<child link = "simple_arm_base_link" />
+		<origin xyz="0.0 0.0 0.0" rpy="0.0 0.0 0.0" />
+	</joint>
+	<xacro:ur3_robot prefix="simple_arm_" joint_limited="true"/>
+	<!-- Robotiq 85-->
+	<xacro:include filename="$(find robotiq_85_description)/urdf/robotiq_85_gripper.urdf.xacro" />
+	<xacro:robotiq_85_gripper prefix="simple_gripper_" parent="simple_arm_tool0">
+		<origin xyz="0 0 0" rpy="${pi/2} -${pi/2} 0" />
+	</xacro:robotiq_85_gripper>
 </robot>

File: ur5_robotiq_85/urdf/ur5_robotiq_85.urdf.xacro (robot description, xacro)
@@ -1,6 +1,19 @@
-<robot name="ur5" xmlns:xacro="http://www.ros.org/wiki/xacro" xmlns:xi="http://www.w3.org/2001/XInclude">
-<!-- combined urdf file -->
-<xacro:include filename="$(find ur_description)/urdf/ur5_robot.urdf.xacro"/>
-<!-- add any joints/links required to connect the two -->
-<xacro:include filename="$(find robotiq_85_description)/urdf/robotiq_85_gripper.xacro" />
+<?xml version="1.0"?>
+<robot name="ur5_robotiq_85" xmlns:xacro="http://ros.org/wiki/xacro">
+	<xacro:arg name="limited" default="true"/>
+	<!-- THE ROBOT -->
+	<link name="world" />
+	<!-- UR5 -->
+	<xacro:include filename="$(find ur_description)/urdf/ur5.urdf.xacro" />
+	<joint name="world_joint" type="fixed">
+		<parent link="world" />
+		<child link = "simple_arm_base_link" />
+		<origin xyz="0.0 0.0 0.0" rpy="0.0 0.0 0.0" />
+	</joint>
+	<xacro:ur5_robot prefix="simple_arm_" joint_limited="true"/>
+	<!-- Robotiq 85-->
+	<xacro:include filename="$(find robotiq_85_description)/urdf/robotiq_85_gripper.urdf.xacro" />
+	<xacro:robotiq_85_gripper prefix="simple_gripper_" parent="simple_arm_tool0">
+		<origin xyz="0 0 0" rpy="${pi/2} -${pi/2} 0" />
+	</xacro:robotiq_85_gripper>
 </robot>
