Commit message: changed fixed frame to base_link

File: ur_description/urdf/ur10_robotiq_85.urdf.xacro (robot description, xacro)
@@ -3,9 +3,9 @@
 	<xacro:arg name="limited" default="true"/>
 	<!-- THE ROBOT -->
-	<link name="base" />
+	<link name="base_link" />
 	<!-- UR10 -->
 	<xacro:include filename="$(find ur_description)/urdf/ur10.urdf.xacro" />
 	<joint name="world_joint" type="fixed">
-		<parent link="base" />
+		<parent link="base_link" />
 		<child link = "simple_arm_base_link" />
 		<origin xyz="0.0 0.0 0.0" rpy="0.0 0.0 0.0" />

File: ur_description/urdf/ur3_robotiq_85.urdf.xacro (robot description, xacro)
@@ -3,9 +3,9 @@
 	<xacro:arg name="limited" default="true"/>
 	<!-- THE ROBOT -->
-	<link name="base" />
+	<link name="base_link" />
 	<!-- UR3 -->
 	<xacro:include filename="$(find ur_description)/urdf/ur3.urdf.xacro" />
 	<joint name="base_joint" type="fixed">
-		<parent link="base" />
+		<parent link="base_link" />
 		<child link = "simple_arm_base_link" />
 		<origin xyz="0.0 0.0 0.0" rpy="0.0 0.0 0.0" />

File: ur_description/urdf/ur5_robotiq_85.urdf.xacro (robot description, xacro)
@@ -3,9 +3,9 @@
 	<xacro:arg name="limited" default="true"/>
 	<!-- THE ROBOT -->
-	<link name="base" />
+	<link name="base_link" />
 	<!-- UR5 -->
 	<xacro:include filename="$(find ur_description)/urdf/ur5.urdf.xacro" />
 	<joint name="world_joint" type="fixed">
-		<parent link="base" />
+		<parent link="base_link" />
 		<child link = "simple_arm_base_link" />
 		<origin xyz="0.0 0.0 0.0" rpy="0.0 0.0 0.0" />

Commit message: removing simple_X_ prefixes from components

File: ur_description/urdf/ur10_robotiq_85.urdf.xacro (robot description, xacro)
@@ -3,16 +3,16 @@
 	<xacro:arg name="limited" default="true"/>
 	<!-- THE ROBOT -->
-	<link name="base_link" />
+	<link name="world" />
 	<!-- UR10 -->
 	<xacro:include filename="$(find ur_description)/urdf/ur10.urdf.xacro" />
 	<joint name="world_joint" type="fixed">
-		<parent link="base_link" />
-		<child link = "simple_arm_base_link" />
+		<parent link="world" />
+		<child link = "base_link" />
 		<origin xyz="0.0 0.0 0.0" rpy="0.0 0.0 0.0" />
 	</joint>
-	<xacro:ur10_robot prefix="simple_arm_" joint_limited="true"/>
+	<xacro:ur10_robot prefix="" joint_limited="true"/>
 	<!-- Robotiq 85-->
 	<xacro:include filename="$(find robotiq_85_description)/urdf/robotiq_85_gripper.urdf.xacro" />
-	<xacro:robotiq_85_gripper prefix="simple_gripper_" parent="simple_arm_tool0">
+	<xacro:robotiq_85_gripper prefix="" parent="tool0">
 		<origin xyz="0 0 0" rpy="${pi/2} -${pi/2} 0" />
 	</xacro:robotiq_85_gripper>

File: ur_description/urdf/ur3_robotiq_85.urdf.xacro (robot description, xacro)
@@ -3,16 +3,16 @@
 	<xacro:arg name="limited" default="true"/>
 	<!-- THE ROBOT -->
-	<link name="base_link" />
+	<link name="world" />
 	<!-- UR3 -->
 	<xacro:include filename="$(find ur_description)/urdf/ur3.urdf.xacro" />
-	<joint name="base_joint" type="fixed">
-		<parent link="base_link" />
-		<child link = "simple_arm_base_link" />
+	<joint name="world_joint" type="fixed">
+		<parent link="world" />
+		<child link = "base_link" />
 		<origin xyz="0.0 0.0 0.0" rpy="0.0 0.0 0.0" />
 	</joint>
-	<xacro:ur3_robot prefix="simple_arm_" joint_limited="true"/>
+	<xacro:ur3_robot prefix="" joint_limited="true"/>
 	<!-- Robotiq 85-->
 	<xacro:include filename="$(find robotiq_85_description)/urdf/robotiq_85_gripper.urdf.xacro" />
-	<xacro:robotiq_85_gripper prefix="simple_gripper_" parent="simple_arm_tool0">
+	<xacro:robotiq_85_gripper prefix="" parent="tool0">
 		<origin xyz="0 0 0" rpy="${pi/2} -${pi/2} 0" />
 	</xacro:robotiq_85_gripper>
