Commit message: updating kinova config

File: robot_description/urdf/kinova_mico/m1n6s.xacro (robot description, xacro)
@@ -135,5 +135,5 @@
           <visual>
             <geometry>
-              <mesh filename="package://m1n6s_robotiq85_moveit_config/meshes/${link_6_mesh}.dae" />
+              <mesh filename="package://robot_descriptions/meshes/kinova_robotiq_coupler/${link_6_mesh}.dae" />
             </geometry>
             <material name="carbon_fiber">
@@ -143,5 +143,5 @@
           <collision>
             <geometry>
-              <mesh filename="package://m1n6s_robotiq85_moveit_config/meshes/${link_6_mesh}.stl" />
+              <mesh filename="package://robot_descriptions/meshes/kinova_robotiq_coupler/${link_6_mesh}.stl" />
             </geometry>
           </collision>
