Commit message: working on relaxed-ik urdfs

File: robot_descriptions/urdf/universal_robots/relaxed_ik_ur5_robotiq_85.urdf.xacro (robot description, xacro)
@@ -3,13 +3,6 @@
 	<xacro:arg name="limited" default="true"/>
 	<!-- THE ROBOT -->
-	<link name="world"/>
 	<!-- UR5 -->
-	<xacro:include filename="$(find ur_description)/urdf/ur5.urdf.xacro" />
-	<joint name="world_joint" type="fixed">
-		<parent link="world" />
-		<child link = "base_link" />
-		<origin xyz="0.0 0.0 0.0" rpy="0.0 0.0 0.0" />
-	</joint>
-	<xacro:ur5_robot prefix="" joint_limited="false"/>
+	<xacro:include filename="$(find robot_descriptions)/urdf/universal_robots/relaxed_ik_ur5.urdf" />
 	<!-- Robotiq 85-->
 	<xacro:include filename="$(find robotiq_85_description)/urdf/robotiq_85_gripper.urdf.xacro" />
