Commit message: adding relaxed-ik configurations

File: relaxed_ik_robot_configs/ur3/ur3.urdf (robot description, URDF)
Before this commit: robot ur5, 11 links, 10 joints
Links:
- link base_link: mass 4.0 -> 2.0; geometry collision mesh filename=package://ur_description/meshes/ur3/collision/base.stl; visual mesh filename=package://ur_description/meshes/ur3/visual/base.dae
- link forearm_link: mass 2.275 -> 1.26; geometry collision mesh filename=package://ur_description/meshes/ur3/collision/forearm.stl; visual mesh filename=package://ur_description/meshes/ur3/visual/forearm.dae
- link shoulder_link: mass 3.7 -> 2.0; geometry collision mesh filename=package://ur_description/meshes/ur3/collision/shoulder.stl; visual mesh filename=package://ur_description/meshes/ur3/visual/shoulder.dae
- link upper_arm_link: mass 8.393 -> 3.42; geometry collision mesh filename=package://ur_description/meshes/ur3/collision/upperarm.stl; visual mesh filename=package://ur_description/meshes/ur3/visual/upperarm.dae
- link wrist_1_link: mass 1.219 -> 0.8; geometry collision mesh filename=package://ur_description/meshes/ur3/collision/wrist1.stl; visual mesh filename=package://ur_description/meshes/ur3/visual/wrist1.dae
- link wrist_2_link: mass 1.219 -> 0.8; geometry collision mesh filename=package://ur_description/meshes/ur3/collision/wrist2.stl; visual mesh filename=package://ur_description/meshes/ur3/visual/wrist2.dae
- link wrist_3_link: mass 0.1879 -> 0.35; geometry collision mesh filename=package://ur_description/meshes/ur3/collision/wrist3.stl; visual mesh filename=package://ur_description/meshes/ur3/visual/wrist3.dae
Joints:
- joint base_link-base_fixed_joint: origin xyz=0 0 0 rpy=0 0 -3.14159265 -> xyz=0 0 0 rpy=0 0 -3.14159265359
- joint ee_fixed_joint: origin xyz=0.0 0.0823 0.0 rpy=0.0 0.0 1.570796325 -> xyz=0.0 0.0819 0.0 rpy=0.0 0.0 1.57079632679
- joint elbow_joint: limit lower=-6.2831853 upper=6.2831853 effort=150.0 velocity=3.15 -> lower=-3.14159265359 upper=3.14159265359 effort=150.0 velocity=3.15; origin xyz=0.0 -0.1197 0.425 rpy=0.0 0.0 0.0 -> xyz=0.0 -0.0925 0.24365 rpy=0.0 0.0 0.0
- joint shoulder_lift_joint: limit lower=-6.2831853 upper=6.2831853 effort=150.0 velocity=3.15 -> lower=-6.28318530718 upper=6.28318530718 effort=330.0 velocity=2.16; origin xyz=0.0 0.13585 0.0 rpy=0.0 0.0 0.0 -> xyz=0.0 0.1198 0.0 rpy=0.0 1.57079632679 0.0
- joint shoulder_pan_joint: limit lower=-6.2831853 upper=6.2831853 effort=150.0 velocity=3.15 -> lower=-6.28318530718 upper=6.28318530718 effort=330.0 velocity=2.16; origin xyz=0.0 0.0 0.089159 rpy=0.0 0.0 0.0 -> xyz=0.0 0.0 0.1519 rpy=0.0 0.0 0.0
- joint wrist_1_joint: limit lower=-6.2831853 upper=6.2831853 effort=28.0 velocity=3.2 -> lower=-6.28318530718 upper=6.28318530718 effort=54.0 velocity=3.2; origin xyz=0.0 0.0 0.39225 rpy=0.0 0.0 0.0 -> xyz=0.0 0.0 0.21325 rpy=0.0 1.57079632679 0.0
- joint wrist_2_joint: limit lower=-6.2831853 upper=6.2831853 effort=28.0 velocity=3.2 -> lower=-6.28318530718 upper=6.28318530718 effort=54.0 velocity=3.2; origin xyz=0.0 0.093 0.0 rpy=0.0 0.0 0.0 -> xyz=0.0 0.08505 0.0 rpy=0.0 0.0 0.0
- joint wrist_3_joint: limit lower=-6.2831853 upper=6.2831853 effort=28.0 velocity=3.2 -> lower=-6.28318530718 upper=6.28318530718 effort=54.0 velocity=3.2; origin xyz=0.0 0.0 0.09465 rpy=0.0 0.0 0.0 -> xyz=0.0 0.0 0.08535 rpy=0.0 0.0 0.0
- joint wrist_3_link-tool0_fixed_joint: origin xyz=0 0.0823 0 rpy=-1.570796325 0 0 -> xyz=0 0.0819 0 rpy=-1.57079632679 0 0

File: robot_descriptions/urdf/kinova_mico/relaxed_ik_m1n6s_robotiq_85.xacro (robot description, xacro)
@@ -1,22 +1,6 @@
 <?xml version="1.0"?>
 <robot name="m1n6s_robotiq85" xmlns:xacro="http://ros.org/wiki/xacro">
-	<link name="root">
-  </link>
-  <!-- for gazebo -->
-  <link name="world"/>
-  <joint name="connect_root_and_world" type="fixed">
-    <child link="root" />
-    <parent link="world" />
-    <origin xyz="0 0 0" rpy="0 0 0" />
-  </joint>
-	<!-- THE ROBOT -->
-	<link name="base_link" />
 	<!-- M1N6S Mico Arm -->
-	<xacro:include filename="$(relaxed_ik_robot_configs)/mico/urdf_mico.xacro" />
-  <joint name="base_joint" type="fixed">
-		<parent link="base_link" />
-		<child link = "root" />
-		<origin xyz="0.0 0.0 0.0" rpy="0.0 0.0 0.0" />
-	</joint>
+	<xacro:include filename="$(relaxed_ik_robot_configs)/mico/mico.urdf" />
 	<!-- Robotiq 85-->
 	<xacro:include filename="$(find robotiq_85_description)/urdf/robotiq_85_gripper.urdf.xacro" />

File: robot_descriptions/urdf/universal_robots/relaxed_ik_ur3_robotiq_85.xacro (robot description, xacro)
@@ -1,8 +1,8 @@
 <?xml version="1.0"?>
-<robot name="ur5_robotiq_85" xmlns:xacro="http://ros.org/wiki/xacro">
+<robot name="ur3_robotiq_85" xmlns:xacro="http://ros.org/wiki/xacro">
 	<xacro:arg name="limited" default="true"/>
 	<!-- THE ROBOT -->
-	<!-- UR5 -->
-	<xacro:include filename="$(find relaxed_ik_robot_configs)/ur5/urdf_ur5.xacro" />
+	<!-- UR3 -->
+	<xacro:include filename="$(find relaxed_ik_robot_configs)/ur3/ur3.urdf" />
 	<!-- Robotiq 85-->
 	<xacro:include filename="$(find robotiq_85_description)/urdf/robotiq_85_gripper.urdf.xacro" />

File: robot_descriptions/urdf/universal_robots/relaxed_ik_ur5_robotiq_85.xacro (robot description, xacro)
@@ -1,8 +1,8 @@
 <?xml version="1.0"?>
-<robot name="ur3_robotiq_85" xmlns:xacro="http://ros.org/wiki/xacro">
+<robot name="ur5_robotiq_85" xmlns:xacro="http://ros.org/wiki/xacro">
 	<xacro:arg name="limited" default="true"/>
 	<!-- THE ROBOT -->
-	<!-- UR3 -->
-	<xacro:include filename="$(find relaxed_ik_robot_configs)/ur3/urdf_ur3.xacro" />
+	<!-- UR5 -->
+	<xacro:include filename="$(find relaxed_ik_robot_configs)/ur5/ur5.urdf" />
 	<!-- Robotiq 85-->
 	<xacro:include filename="$(find robotiq_85_description)/urdf/robotiq_85_gripper.urdf.xacro" />
